File: PCB/Main board v1.kicad_sch (KiCad schematic)
At the start: 2 parts, among them J1 Conn_01x22_Socket, J2 Conn_01x22_Socket

Commit message: restructure
Connections:
- net +3V3: no longer J1.2 (Pin_2)
- net GND: no longer J2.1 (Pin_1), J2.2 (Pin_2)
Changed lines of the file:
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@@
 	(generator_version "9.0")
 	(paper "A4")
-	(junction
-		(at 129.54 39.37)
-		(diameter 0)
-		(color 0 0 0 0)
-	)
-	(junction
-		(at 163.83 92.71)
-		(diameter 0)
-		(color 0 0 0 0)
-	)
-	(wire
-		(pts
-			(xy 129.54 39.37) (xy 129.54 41.91)
-		)
-		(stroke
-			(width 0)
-			(type default)
-		)
-	)
-	(wire
-		(pts
-			(xy 161.29 90.17) (xy 163.83 90.17)
-		)
-		(stroke
-			(width 0)
-			(type default)
-		)
-	)
 	(wire
 		(pts
@@
 	(wire
 		(pts
-			(xy 163.83 90.17) (xy 163.83 92.71)
-		)
-		(stroke
-			(width 0)
-			(type default)
-		)
-	)
-	(wire
-		(pts
 			(xy 129.54 90.17) (xy 132.08 90.17)
 		)
@@
 	(wire
 		(pts
-			(xy 129.54 41.91) (xy 132.08 41.91)
-		)
-		(stroke
-			(width 0)
-			(type default)
-		)
-	)
-	(wire
-		(pts
 			(xy 129.54 38.1) (xy 129.54 39.37)
 		)
@@
 		(pts
 			(xy 161.29 39.37) (xy 163.83 39.37)
-		)
-		(stroke
-			(width 0)
-			(type default)
-		)
-	)
-	(wire
-		(pts
-			(xy 161.29 92.71) (xy 163.83 92.71)
 		)
 		(stroke
@@
 					(unit 1)
 				)
-			)
-		)
-	)
-	(symbol
-		(lib_id "power:GND")
-		(at 163.83 92.71 0)
-		(unit 1)
-		(exclude_from_sim no)
-		(in_bom yes)
-		(on_board yes)
-		(dnp no)
-		(property "Reference" "#PWR04"
-			(at 163.83 99.06 0)
-			(effects
-				(font
-					(size 1.27 1.27)
-				)
-				(hide yes)
-			)
-		)
-		(property "Value" "GND"
-			(at 167.132 96.012 0)
-			(effects
-				(font
-					(size 1.27 1.27)
-				)
-			)
-		)
-		(property "Footprint" ""
-			(at 163.83 92.71 0)
-			(effects
-				(font
-					(size 1.27 1.27)
-				)
-				(hide yes)
-			)
-		)
-		(property "Datasheet" ""
-			(at 163.83 92.71 0)
-			(effects
-				(font
-					(size 1.27 1.27)
-				)
-				(hide yes)
-			)
-		)
-		(property "Description" "Power symbol creates a global label with name \"GND\" , ground"
-			(at 163.83 92.71 0)
-			(effects
-				(font
-					(size 1.27 1.27)
-				)
-				(hide yes)
-			)
-		)
-		(pin "1"
-		)
-		(instances
-			(project "PCB - main board v1"
-				(path "/5fb6f33a-61ea-485d-8e93-d2d4429c2b7d"
-					(reference "#PWR04")
-					(unit 1)
-				)
